File: kicad/tutorial1/tutorial1.sch (KiCad schematic (older format))
At the start: 3 parts

Commit message: before layerd
Parts:
- removed D?: LED, symbol Device:LED
- removed R?: R, symbol Device:R
- removed U?: PIC12C508A-ISN, Package_DIP:DIP-8_W7.62mm, symbol MCU_Microchip_PIC12:PIC12C508A-ISN
- added C1: CP, symbol Device:CP
- added C2, C3: C, symbol Device:C
- added CN1, CN2: Conn_01x10, symbol Connector_Generic:Conn_01x10
- added CN3: Conn_02x5, symbol Connector_Generic:Conn_01x10
- added D1, D2, D3, D4, D5, D6, D7, D8: LED, symbol Device:LED
- added Q1, Q2, Q3, Q4, Q5, Q6, Q7, Q8: BS170, Package_TO_SOT_THT:TO-92_Inline, symbol Transistor_FET:BS170
- added R1, R2, R3, R4, R5, R6, R7, R8: R, symbol Device:R
- added RN1, RN2: R_Network08, Resistor_THT:R_Array_SIP9, symbol Device:R_Network08
- added RV1: R_POT_TRIM, symbol Device:R_POT_TRIM
- added SW1, SW2: SW_DIP_x08, symbol Switch:SW_DIP_x08
Connections:
- net labels added: +5V
- net labels removed: VCC
- wire segments 11 -> 156
