File: kicad/tutorial1/tutorial1.sch (KiCad schematic (older format))
At the start: 35 parts, among them CN1 Conn_01x10, CN2 Conn_01x10, CN3 Conn_02x5, Q1 BS170, Q2 BS170, Q3 BS170, Q4 BS170, Q5 BS170, Q6 BS170, Q7 BS170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

Commit message: kicad
Parts:
- C1: footprint (none) -> My_Device:CP_Radial_D5.0mm_P2.00mm
- C2, C3: footprint (none) -> My_Device:C_Disc_D5.0mm_W2.5mm_P2.50mm
- CN1, CN2, CN3: footprint (none) -> My_Device:BH-10SG
- D1, D2, D3, D4, D5, D6, D7, D8: footprint (none) -> My_Device:LED_D3.0mm
- R1, R2, R3, R4, R5, R6, R7, R8: footprint (none) -> My_Device:R_250mWmono-STD
- RV1: footprint (none) -> My_Device:Potentiometer_Vishay_148-149_Single_Horizontal
- SW1, SW2: footprint (none) -> My_Device:SW_DIP_x8_W7.62mm_Slide
Changed lines of the file:
@@
 F 0 "CN1" V 3367 1296 50  0000 C CNN
 F 1 "Conn_01x10" V 3276 1296 50  0000 C CNN
-F 2 "" H 3150 1350 50  0001 C CNN
+F 2 "My_Device:BH-10SG" H 3150 1350 50  0001 C CNN
 F 3 "~" H 3150 1350 50  0001 C CNN
 	1    3150 1350
@@
 F 0 "SW1" V 3104 5280 50  0000 L CNN
 F 1 "SW_DIP_x08" V 3195 5280 50  0000 L CNN
-F 2 "" H 3150 4750 50  0001 C CNN
+F 2 "My_Device:SW_DIP_x8_W7.62mm_Slide" H 3150 4750 50  0001 C CNN
 F 3 "~" H 3150 4750 50  0001 C CNN
 	1    3150 4750
@@
 F 0 "CN2" V 6567 1296 50  0000 C CNN
 F 1 "Conn_01x10" V 6476 1296 50  0000 C CNN
-F 2 "" H 6350 1350 50  0001 C CNN
+F 2 "My_Device:BH-10SG" H 6350 1350 50  0001 C CNN
 F 3 "~" H 6350 1350 50  0001 C CNN
 	1    6350 1350
@@
 F 0 "R3" H 5870 5046 50  0000 L CNN
 F 1 "R" H 5870 4955 50  0000 L CNN
-F 2 "" V 5730 5000 50  0001 C CNN
+F 2 "My_Device:R_250mWmono-STD" V 5730 5000 50  0001 C CNN
 F 3 "~" H 5800 5000 50  0001 C CNN
 	1    5800 5000
@@
 F 0 "D4" V 6339 4578 50  0000 L CNN
 F 1 "LED" V 6248 4578 50  0000 L CNN
-F 2 "" H 6300 4500 50  0001 C CNN
+F 2 "My_Device:LED_D3.0mm" H 6300 4500 50  0001 C CNN
 F 3 "~" H 6300 4500 50  0001 C CNN
 	1    6300 4500
@@
 F 0 "R4" H 6370 5046 50  0000 L CNN
 F 1 "R" H 6370 4955 50  0000 L CNN
-F 2 "" V 6230 5000 50  0001 C CNN
+F 2 "My_Device:R_250mWmono-STD" V 6230 5000 50  0001 C CNN
 F 3 "~" H 6300 5000 50  0001 C CNN
 	1    6300 5000
@@
 F 0 "D5" V 6839 4578 50  0000 L CNN
 F 1 "LED" V 6748 4578 50  0000 L CNN
-F 2 "" H 6800 4500 50  0001 C CNN
+F 2 "My_Device:LED_D3.0mm" H 6800 4500 50  0001 C CNN
 F 3 "~" H 6800 4500 50  0001 C CNN
 	1    6800 4500
@@
 F 0 "R5" H 6870 5046 50  0000 L CNN
 F 1 "R" H 6870 4955 50  0000 L CNN
-F 2 "" V 6730 5000 50  0001 C CNN
+F 2 "My_Device:R_250mWmono-STD" V 6730 5000 50  0001 C CNN
 F 3 "~" H 6800 5000 50  0001 C CNN
 	1    6800 5000
@@
 F 0 "D6" V 7339 4578 50  0000 L CNN
 F 1 "LED" V 7248 4578 50  0000 L CNN
-F 2 "" H 7300 4500 50  0001 C CNN
+F 2 "My_Device:LED_D3.0mm" H 7300 4500 50  0001 C CNN
 F 3 "~" H 7300 4500 50  0001 C CNN
 	1    7300 4500
@@
 F 0 "R6" H 7370 5046 50  0000 L CNN
 F 1 "R" H 7370 4955 50  0000 L CNN
-F 2 "" V 7230 5000 50  0001 C CNN
+F 2 "My_Device:R_250mWmono-STD" V 7230 5000 50  0001 C CNN
 F 3 "~" H 7300 5000 50  0001 C CNN
 	1    7300 5000
@@
 F 0 "D7" V 7839 4578 50  0000 L CNN
 F 1 "LED" V 7748 4578 50  0000 L CNN
-F 2 "" H 7800 4500 50  0001 C CNN
+F 2 "My_Device:LED_D3.0mm" H 7800 4500 50  0001 C CNN
 F 3 "~" H 7800 4500 50  0001 C CNN
 	1    7800 4500
@@
 F 0 "R7" H 7870 5046 50  0000 L CNN
 F 1 "R" H 7870 4955 50  0000 L CNN
-F 2 "" V 7730 5000 50  0001 C CNN
+F 2 "My_Device:R_250mWmono-STD" V 7730 5000 50  0001 C CNN
 F 3 "~" H 7800 5000 50  0001 C CNN
 	1    7800 5000
@@
 F 0 "D8" V 8339 4578 50  0000 L CNN
 F 1 "LED" V 8248 4578 50  0000 L CNN
-F 2 "" H 8300 4500 50  0001 C CNN
+F 2 "My_Device:LED_D3.0mm" H 8300 4500 50  0001 C CNN
 F 3 "~" H 8300 4500 50  0001 C CNN
 	1    8300 4500
@@
 F 0 "R8" H 8370 5046 50  0000 L CNN
 F 1 "R" H 8370 4955 50  0000 L CNN
-F 2 "" V 8230 5000 50  0001 C CNN
+F 2 "My_Device:R_250mWmono-STD" V 8230 5000 50  0001 C CNN
 F 3 "~" H 8300 5000 50  0001 C CNN
 	1    8300 5000
@@
 F 0 "D3" V 5839 4578 50  0000 L CNN
 F 1 "LED" V 5748 4578 50  0000 L CNN
-F 2 "" H 5800 4500 50  0001 C CNN
+F 2 "My_Device:LED_D3.0mm" H 5800 4500 50  0001 C CNN
 F 3 "~" H 5800 4500 50  0001 C CNN
 	1    5800 4500
@@
 F 0 "R2" H 5370 5046 50  0000 L CNN
 F 1 "R" H 5370 4955 50  0000 L CNN
-F 2 "" V 5230 5000 50  0001 C CNN
+F 2 "My_Device:R_250mWmono-STD" V 5230 5000 50  0001 C CNN
 F 3 "~" H 5300 5000 50  0001 C CNN
 	1    5300 5000
@@
 F 0 "D2" V 5339 4578 50  0000 L CNN
 F 1 "LED" V 5248 4578 50  0000 L CNN
-F 2 "" H 5300 4500 50  0001 C CNN
+F 2 "My_Device:LED_D3.0mm" H 5300 4500 50  0001 C CNN
 F 3 "~" H 5300 4500 50  0001 C CNN
 	1    5300 4500
@@
 F 0 "R1" H 4870 5046 50  0000 L CNN
 F 1 "R" H 4870 4955 50  0000 L CNN
-F 2 "" V 4730 5000 50  0001 C CNN
+F 2 "My_Device:R_250mWmono-STD" V 4730 5000 50  0001 C CNN
 F 3 "~" H 4800 5000 50  0001 C CNN
 	1    4800 5000
@@
 F 0 "D1" V 4839 4578 50  0000 L CNN
 F 1 "LED" V 4748 4578 50  0000 L CNN
-F 2 "" H 4800 4500 50  0001 C CNN
+F 2 "My_Device:LED_D3.0mm" H 4800 4500 50  0001 C CNN
 F 3 "~" H 4800 4500 50  0001 C CNN
 	1    4800 4500
@@
 F 0 "CN3" V 9867 1296 50  0000 C CNN
 F 1 "Conn_02x5" V 9776 1296 50  0000 C CNN
-F 2 "" H 9650 1350 50  0001 C CNN
+F 2 "My_Device:BH-10SG" H 9650 1350 50  0001 C CNN
 F 3 "~" H 9650 1350 50  0001 C CNN
 	1    9650 1350
@@
 F 0 "SW2" V 9604 2630 50  0000 L CNN
 F 1 "SW_DIP_x08" V 9695 2630 50  0000 L CNN
-F 2 "" H 9650 2100 50  0001 C CNN
+F 2 "My_Device:SW_DIP_x8_W7.62mm_Slide" H 9650 2100 50  0001 C CNN
 F 3 "~" H 9650 2100 50  0001 C CNN
 	1    9650 2100
@@
 F 0 "C3" H 10165 2846 50  0000 L CNN
 F 1 "C" H 10165 2755 50  0000 L CNN
-F 2 "" H 10088 2650 50  0001 C CNN
+F 2 "My_Device:C_Disc_D5.0mm_W2.5mm_P2.50mm" H 10088 2650 50  0001 C CNN
 F 3 "~" H 10050 2800 50  0001 C CNN
 	1    10050 2800
@@
 F 0 "RV1" H 10330 2696 50  0000 R CNN
 F 1 "R_POT_TRIM" H 10330 2605 50  0000 R CNN
-F 2 "" H 10400 2650 50  0001 C CNN
+F 2 "My_Device:Potentiometer_Vishay_148-149_Single_Horizontal" H 10400 2650 50  0001 C CNN
 F 3 "~" H 10400 2650 50  0001 C CNN
 	1    10400 2650
@@
 F 0 "C1" H 9968 4246 50  0000 L CNN
 F 1 "CP" H 9968 4155 50  0000 L CNN
-F 2 "" H 9888 4050 50  0001 C CNN
+F 2 "My_Device:CP_Radial_D5.0mm_P2.00mm" H 9888 4050 50  0001 C CNN
 F 3 "~" H 9850 4200 50  0001 C CNN
 	1    9850 4200
@@
 F 0 "C2" H 10365 4246 50  0000 L CNN
 F 1 "C" H 10365 4155 50  0000 L CNN
-F 2 "" H 10288 4050 50  0001 C CNN
+F 2 "My_Device:C_Disc_D5.0mm_W2.5mm_P2.50mm" H 10288 4050 50  0001 C CNN
 F 3 "~" H 10250 4200 50  0001 C CNN
 	1    10250 4200

Commit message: haisen
Connections:
- net +5V: now also D1.2 (A), D2.2 (A), D3.2 (A), D4.2 (A), D5.2 (A), D6.2 (A), D7.2 (A), D8.2 (A)
Changed lines of the file:
@@
 Wire Wire Line
 	3550 4250 3550 4450
+$Comp
+L power:+5V #PWR?
+U 1 1 6394A1B9
+P 8300 4150
+F 0 "#PWR?" H 8300 4000 50  0001 C CNN
+F 1 "+5V" H 8315 4323 50  0000 C CNN
+F 2 "" H 8300 4150 50  0001 C CNN
+F 3 "" H 8300 4150 50  0001 C CNN
+	1    8300 4150
+	1    0    0    -1
+$EndComp
+Wire Wire Line
+	8300 4150 8300 4350
+Connection ~ 8300 4350
 $EndSCHEMATC

Commit message: before net apply
Parts:
- added U1: bord, My_Device:pcb_100x75mm, symbol My_device:bord
Changed lines of the file:
@@
 	3550 4250 3550 4450
 $Comp
-L power:+5V #PWR?
+L power:+5V #PWR0101
 U 1 1 6394A1B9
 P 8300 4150
-F 0 "#PWR?" H 8300 4000 50  0001 C CNN
+F 0 "#PWR0101" H 8300 4000 50  0001 C CNN
 F 1 "+5V" H 8315 4323 50  0000 C CNN
 F 2 "" H 8300 4150 50  0001 C CNN
@@
 	8300 4150 8300 4350
 Connection ~ 8300 4350
+$Comp
+L My_device:bord U1
+U 1 1 6398D3A2
+P 10400 5850
+F 0 "U1" H 10650 5938 50  0000 L CNN
+F 1 "bord" H 10650 5847 50  0000 L CNN
+F 2 "My_Device:pcb_100x75mm" H 10400 5850 50  0001 C CNN
+F 3 "" H 10400 5850 50  0001 C CNN
+	1    10400 5850
+	1    0    0    -1
+$EndComp
 $EndSCHEMATC
