File: kicad/tutorial1/tutorial1.kicad_pcb (KiCad board)
At the start: 2 copper layers, 35 parts, among them CN1 Conn_01x10, CN2 Conn_01x10, CN3 Conn_02x5, Q1 BS170, Q2 BS170, Q3 BS170, Q4 BS170, Q5 BS170, Q6 BS170, Q7 BS170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

Commit message: before net apply
Parts:
- added U1: bord, My_Device:pcb_100x75mm, F.Cu at (151.9, 76.8)
- moved D3 160.3 mm to (191.3, 83.1)
- moved D7 160.3 mm to (191.3, 88.7)
- moved D2 160.3 mm to (178.3, 89.7)
- moved D5 160.3 mm to (184.2, 89.7)
- moved D6 160.3 mm to (178.3, 95.3)
- moved D8 160.3 mm to (184.2, 95.3)
- moved Q5 160.3 mm to (185.1, 84.4)
- moved Q6 160.3 mm to (178.6, 84.4)
- moved CN2 160.2 mm to (165.3, 95.9)
- moved D1 146.4 mm to (113.7, 104.2)
- moved Q3 146.4 mm to (120.5, 104.3)
- moved Q4 146.4 mm to (127.0, 104.3)
- moved Q8 146.4 mm to (133.5, 104.3)
- moved Q7 146.4 mm to (140.0, 104.3)
- moved CN1 146.2 mm to (188.9, 56.7)
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Changed lines of the file:
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@@
     (tracks 0)
     (zones 0)
-    (modules 35)
+    (modules 36)
     (nets 44)
   )
@@
     (pad_to_mask_clearance 0.051)
     (solder_mask_min_width 0.25)
-    (aux_axis_origin 0 0)
+    (aux_axis_origin 101.854 114.292)
+    (grid_origin 101.854 114.292)
     (visible_elements 7FFFFFFF)
     (pcbplotparams
@@
     (add_net "Net-(Q8-Pad1)")
   )
+  (module My_Device:pcb_100x75mm (layer F.Cu)
+    (at 151.854 76.792)
+    (fp_text reference U1 (at -0.3691 -35.9792 180) (layer F.SilkS) hide
+      (effects (font (size 1 1) (thickness 0.15)))
+    )
+    (fp_text value bord (at -0.2591 -35.0492 180) (layer F.Fab) hide
+      (effects (font (size 1 1) (thickness 0.15)))
+    )
+    (fp_line (start 50 -37.5) (end 50 37.5) (layer F.CrtYd) (width 0.05))
+    (fp_line (start -50 -37.5) (end 50 -37.5) (layer F.CrtYd) (width 0.05))
+    (fp_line (start -50 37.5) (end -50 -37.5) (layer F.CrtYd) (width 0.05))
+    (fp_line (start 50 37.5) (end -50 37.5) (layer F.CrtYd) (width 0.05))
+    (pad "" np_thru_hole circle (at 46 -33.5 90) (size 6 6) (drill 3.2) (layers *.Cu *.Mask))
+    (pad "" np_thru_hole circle (at 45 32.5 90) (size 6 6) (drill 3.2) (layers *.Cu *.Mask))
+    (pad "" np_thru_hole circle (at -46 33.5 90) (size 6 6) (drill 3.2) (layers *.Cu *.Mask))
+    (pad "" np_thru_hole circle (at -46 -33.5 90) (size 6 6) (drill 3.2) (layers *.Cu *.Mask))
+  )
   (module My_Device:SW_DIP_x8_W7.62mm_Slide (layer F.Cu)
-    (at 12.915225 -8.735)
+    (at 136.769225 53.057)
     (descr "8x-dip-switch, Slide, row spacing 7.62 mm (300 mils)")
     (tags "DIP Switch Slide 7.62mm 300mil")
@@
   )
   (module My_Device:SW_DIP_x8_W7.62mm_Slide (layer F.Cu)
-    (at -11.884775 -0.035)
+    (at 111.969225 61.757)
     (descr "8x-dip-switch, Slide, row spacing 7.62 mm (300 mils)")
     (tags "DIP Switch Slide 7.62mm 300mil")
@@
   )
   (module My_Device:Potentiometer_Vishay_148-149_Single_Horizontal (layer F.Cu)
-    (at 2.160225 21.76)
+    (at 126.014225 83.552)
     (descr "Potentiometer, horizontal, Vishay 148-149 Single, http://www.vishay.com/docs/57040/148149.pdf")
     (tags "Potentiometer horizontal Vishay 148-149 Single")
@@
   )
   (module Resistor_THT:R_Array_SIP9 (layer F.Cu)
-    (at -11.619775 -9.8)
+    (at 112.234225 51.992)
     (descr "9-pin Resistor SIP pack")
     (tags R)
@@
   )
   (module Resistor_THT:R_Array_SIP9 (layer F.Cu)
-    (at -11.619775 -5.45)
+    (at 112.234225 56.342)
     (descr "9-pin Resistor SIP pack")
     (tags R)
@@
   )
   (module My_Device:R_250mWmono-STD (layer F.Cu)
-    (at 26.217224 -11.225001)
+    (at 150.071224 50.566999)
     (fp_text reference R8 (at 0 0.5) (layer F.SilkS)
       (effects (font (size 1 1) (thickness 0.15)))
@@
   )
   (module My_Device:R_250mWmono-STD (layer F.Cu)
-    (at 28.737224 -11.225001)
+    (at 152.591224 50.566999)
     (fp_text reference R7 (at 0 0.5) (layer F.SilkS)
       (effects (font (size 1 1) (thickness 0.15)))
@@
   )
   (module My_Device:R_250mWmono-STD (layer F.Cu)
-    (at 31.257224 -11.225001)
+    (at 155.111224 50.566999)
     (fp_text reference R6 (at 0 0.5) (layer F.SilkS)
       (effects (font (size 1 1) (thickness 0.15)))
@@
   )
   (module My_Device:R_250mWmono-STD (layer F.Cu)
-    (at 23.697224 -11.225001)
+    (at 147.551224 50.566999)
     (fp_text reference R5 (at 0 0.5) (layer F.SilkS)
       (effects (font (size 1 1) (thickness 0.15)))
@@
   )
   (module My_Device:R_250mWmono-STD (layer F.Cu)
-    (at 33.777224 -11.225001)
+    (at 157.631224 50.566999)
     (fp_text reference R4 (at 0 0.5) (layer F.SilkS)
       (effects (font (size 1 1) (thickness 0.15)))
@@
   )
   (module My_Device:R_250mWmono-STD (layer F.Cu)
-    (at 36.297224 -11.225001)
+    (at 160.151224 50.566999)
     (fp_text reference R3 (at 0 0.5) (layer F.SilkS)
       (effects (font (size 1 1) (thickness 0.15)))
@@
   )
   (module My_Device:R_250mWmono-STD (layer F.Cu)
-    (at 38.817224 -11.225001)
+    (at 162.671224 50.566999)
     (fp_text reference R2 (at 0 0.5) (layer F.SilkS)
       (effects (font (size 1 1) (thickness 0.15)))
@@
   )
   (module My_Device:R_250mWmono-STD (layer F.Cu)
-    (at 41.337224 -11.225001)
+    (at 165.191224 50.566999)
     (fp_text reference R1 (at 0 0.5) (layer F.SilkS)
       (effects (font (size 1 1) (thickness 0.15)))
@@
   )
   (module Package_TO_SOT_THT:TO-92_Inline (layer F.Cu)
-    (at 7.670225 29.54)
+    (at 133.524225 104.332)
     (descr "TO-92 leads in-line, narrow, oval pads, drill 0.75mm (see NXP sot054_po.pdf)")
     (tags "to-92 sc-43 sc-43a sot54 PA33 transistor")
@@
   )
   (module Package_TO_SOT_THT:TO-92_Inline (layer F.Cu)
-    (at 14.180225 29.54)
+    (at 140.034225 104.332)
     (descr "TO-92 leads in-line, narrow, oval pads, drill 0.75mm (see NXP sot054_po.pdf)")
     (tags "to-92 sc-43 sc-43a sot54 PA33 transistor")
@@
   )
   (module Package_TO_SOT_THT:TO-92_Inline (layer F.Cu)
-    (at 34.770225 13.61)
+    (at 178.624225 84.402)
     (descr "TO-92 leads in-line, narrow, oval pads, drill 0.75mm (see NXP sot054_po.pdf)")
     (tags "to-92 sc-43 sc-43a sot54 PA33 transistor")
@@
   )
   (module Package_TO_SOT_THT:TO-92_Inline (layer F.Cu)
-    (at 41.280225 13.61)
+    (at 185.134225 84.402)
     (descr "TO-92 leads in-line, narrow, oval pads, drill 0.75mm (see NXP sot054_po.pdf)")
     (tags "to-92 sc-43 sc-43a sot54 PA33 transistor")
@@
   )
   (module Package_TO_SOT_THT:TO-92_Inline (layer F.Cu)
-    (at 1.160225 29.54)
+    (at 127.014225 104.332)
     (descr "TO-92 leads in-line, narrow, oval pads, drill 0.75mm (see NXP sot054_po.pdf)")
     (tags "to-92 sc-43 sc-43a sot54 PA33 transistor")
@@
   )
   (module Package_TO_SOT_THT:TO-92_Inline (layer F.Cu)
-    (at -5.349775 29.54)
+    (at 120.504225 104.332)
     (descr "TO-92 leads in-line, narrow, oval pads, drill 0.75mm (see NXP sot054_po.pdf)")
     (tags "to-92 sc-43 sc-43a sot54 PA33 transistor")
@@
   )
   (module Package_TO_SOT_THT:TO-92_Inline (layer F.Cu)
-    (at 6.250225 4.03)
+    (at 130.104225 65.822)
     (descr "TO-92 leads in-line, narrow, oval pads, drill 0.75mm (see NXP sot054_po.pdf)")
     (tags "to-92 sc-43 sc-43a sot54 PA33 transistor")
@@
   )
   (module Package_TO_SOT_THT:TO-92_Inline (layer F.Cu)
-    (at -11.859775 24.14)
+    (at 111.994225 85.932)
     (descr "TO-92 leads in-line, narrow, oval pads, drill 0.75mm (see NXP sot054_po.pdf)")
     (tags "to-92 sc-43 sc-43a sot54 PA33 transistor")
@@
   )
   (module My_Device:LED_D3.0mm (layer F.Cu)
-    (at 40.360225 24.47)
+    (at 184.214225 95.262)
     (descr "LED, diameter 3.0mm, 2 pins")
     (tags "LED diameter 3.0mm 2 pins")
@@
   )
   (module My_Device:LED_D3.0mm (layer F.Cu)
-    (at 47.480225 17.9)
+    (at 191.334225 88.692)
     (descr "LED, diameter 3.0mm, 2 pins")
     (tags "LED diameter 3.0mm 2 pins")
@@
   )
   (module My_Device:LED_D3.0mm (layer F.Cu)
-    (at 34.460225 24.47)
+    (at 178.314225 95.262)
     (descr "LED, diameter 3.0mm, 2 pins")
     (tags "LED diameter 3.0mm 2 pins")
@@
   )
   (module My_Device:LED_D3.0mm (layer F.Cu)
-    (at 40.360225 18.92)
+    (at 184.214225 89.712)
     (descr "LED, diameter 3.0mm, 2 pins")
     (tags "LED diameter 3.0mm 2 pins")
@@
   )
   (module My_Device:LED_D3.0mm (layer F.Cu)
-    (at 5.860225 9.34)
+    (at 129.714225 71.132)
     (descr "LED, diameter 3.0mm, 2 pins")
     (tags "LED diameter 3.0mm 2 pins")
@@
   )
   (module My_Device:LED_D3.0mm (layer F.Cu)
-    (at 47.480225 12.35)
+    (at 191.334225 83.142)
     (descr "LED, diameter 3.0mm, 2 pins")
     (tags "LED diameter 3.0mm 2 pins")
@@
   )
   (module My_Device:LED_D3.0mm (layer F.Cu)
-    (at 34.460225 18.92)
+    (at 178.314225 89.712)
     (descr "LED, diameter 3.0mm, 2 pins")
     (tags "LED diameter 3.0mm 2 pins")
@@
   )
   (module My_Device:LED_D3.0mm (layer F.Cu)
-    (at -12.169775 29.45)
+    (at 113.684225 104.242)
     (descr "LED, diameter 3.0mm, 2 pins")
     (tags "LED diameter 3.0mm 2 pins")
@@
   )
   (module My_Device:BH-10SG (layer F.Cu)
-    (at 46.520225 -6.25)
+    (at 170.374225 55.542)
     (fp_text reference CN3 (at 0 -7.12) (layer F.SilkS)
       (effects (font (size 1 1) (thickness 0.15)))
@@
   )
   (module My_Device:BH-10SG (layer F.Cu)
-    (at 26.360225 16.08)
+    (at 165.314 95.872)
     (fp_text reference CN2 (at 0 -7.12) (layer F.SilkS)
       (effects (font (size 1 1) (thickness 0.15)))
@@
   )
   (module My_Device:BH-10SG (layer F.Cu)
-    (at 56.870225 -6.25)
+    (at 188.854 56.712)
     (fp_text reference CN1 (at 0 -7.12) (layer F.SilkS)
       (effects (font (size 1 1) (thickness 0.15)))
@@
   )
   (module My_Device:C_Disc_D5.0mm_W2.5mm_P2.50mm (layer F.Cu)
-    (at -0.339775 5.3)
+    (at 123.514225 67.092)
     (descr "C, Disc series, Radial, pin pitch=2.50mm, , diameter*width=5*2.5mm^2, Capacitor, http://cdn-reichelt.de/documents/datenblatt/B300/DS_KERKO_TC.pdf")
     (tags "C Disc series Radial pin pitch 2.50mm  diameter 5mm width 2.5mm Capacitor")
@@
   )
   (module My_Device:C_Disc_D5.0mm_W2.5mm_P2.50mm (layer F.Cu)
-    (at 6.290225 -1.25)
+    (at 130.144225 60.542)
     (descr "C, Disc series, Radial, pin pitch=2.50mm, , diameter*width=5*2.5mm^2, Capacitor, http://cdn-reichelt.de/documents/datenblatt/B300/DS_KERKO_TC.pdf")
     (tags "C Disc series Radial pin pitch 2.50mm  diameter 5mm width 2.5mm Capacitor")
@@
   )
   (module My_Device:CP_Radial_D5.0mm_P2.00mm (layer F.Cu)
-    (at 0 0)
+    (at 123.854 61.792)
     (descr "CP, Radial series, Radial, pin pitch=2.00mm, , diameter=5mm, Electrolytic Capacitor")
     (tags "CP Radial series Radial pin pitch 2.00mm  diameter 5mm Electrolytic Capacitor")

Commit message: after net and ground
Routing:
- added copper zone on B.Cu, net GND
- added copper zone on F.Cu, net GND
Changed lines of the file:
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@@
   (page A4)
   (layers
-    (0 F.Cu signal)
+    (0 F.Cu signal hide)
     (31 B.Cu signal)
     (32 B.Adhes user)
@@
     )
   )
+  (zone (net 1) (net_name GND) (layer F.Cu) (hatch edge 0.508)
+    (connect_pads (clearance 0.35))
+    (min_thickness 0.254)
+    (fill (arc_segments 32) (thermal_gap 0.508) (thermal_bridge_width 0.508))
+    (polygon
+      (pts
+        (xy 102.362 113.784) (xy 201.422 113.784) (xy 201.422 39.616) (xy 102.362 39.616)
+      )
+    )
+  )
+  (zone (net 1) (net_name GND) (layer B.Cu) (hatch edge 0.508)
+    (connect_pads (clearance 0.35))
+    (min_thickness 0.254)
+    (fill (arc_segments 32) (thermal_gap 0.508) (thermal_bridge_width 0.508))
+    (polygon
+      (pts
+        (xy 102.362 113.784) (xy 201.422 113.784) (xy 201.422 39.616) (xy 102.362 39.616)
+      )
+    )
+  )

Commit message: pcb
Parts:
- moved CN1 115.7 mm to (80.8, 15.5), turned to 180 degrees
- moved RN2 113.5 mm to (95.2, -60.2)
- moved C3 108.2 mm to (182.9, -23.4), turned to 180 degrees
- moved SW2 106.1 mm to (143.3, -52.8), turned to 90 degrees
- moved RN1 104.5 mm to (56.9, -32.3)
- moved SW1 99.2 mm to (33.0, 1.77), turned to 180 degrees
- moved CN3 95.2 mm to (158.0, -38.9), turned to 270 degrees
- moved C2 94.7 mm to (174.0, -23.4)
- moved Q1 79.4 mm to (33.3, 75.4)
- moved RV1 67.0 mm to (63.2, 60.2)
- moved C1 57.1 mm to (98.0, 10.9)
- moved Q7 42.8 mm to (132.8, 146.6)
- moved Q8 42.7 mm to (127.0, 146.6)
- moved Q4 42.7 mm to (120.9, 146.6)
- moved Q3 42.6 mm to (114.8, 146.6)
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